File: breadboard-hole-test.brd (EAGLE design)
At the start: 457.2 x 393.7 mm, 0 parts

Commit message: prototype 3 as cut
Other:
- board size 457.2 x 393.7 mm -> 591.6 x 420.1 mm
- board text added: ".25"
- board text added: ".28"
- board text added: ".3"
- board text added: ".32"
- board text added: ".328"
