File: paint-stencil.brd (EAGLE design)
At the start: 457.2 x 393.7 mm, 0 parts

Commit message: a few tweaks to things
Routing:
- net S$4: track 754.4 -> 0.00 mm
- net S$2: track 754.4 -> 0.00 mm
Changed lines of the file:
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@@
 <layer number="18" name="Vias" color="2" fill="1" visible="no" active="yes"/>
 <layer number="19" name="Unrouted" color="6" fill="1" visible="no" active="yes"/>
-<layer number="20" name="Dimension" color="15" fill="1" visible="yes" active="yes"/>
-<layer number="21" name="tPlace" color="16" fill="1" visible="no" active="yes"/>
+<layer number="20" name="Dimension" color="10" fill="1" visible="yes" active="yes"/>
+<layer number="21" name="tPlace" color="9" fill="1" visible="yes" active="yes"/>
 <layer number="22" name="bPlace" color="14" fill="1" visible="no" active="yes"/>
 <layer number="23" name="tOrigins" color="15" fill="1" visible="no" active="yes"/>
@@
 <wire x1="393.192" y1="355.6" x2="394.208" y2="355.6" width="0.2032" layer="51"/>
 <wire x1="393.7" y1="355.092" x2="393.7" y2="356.108" width="0.2032" layer="51"/>
+<circle x="12.7" y="0" radius="4.5085" width="0.2032" layer="16"/>
+<circle x="127" y="0" radius="4.5085" width="0.2032" layer="1"/>
+<circle x="127" y="177.8" radius="4.5085" width="0.2032" layer="1"/>
+<circle x="127" y="355.6" radius="4.5085" width="0.2032" layer="1"/>
+<circle x="304.8" y="355.6" radius="4.5085" width="0.2032" layer="1"/>
+<circle x="304.8" y="177.8" radius="4.5085" width="0.2032" layer="1"/>
+<circle x="304.8" y="0" radius="4.5085" width="0.2032" layer="1"/>
+<circle x="12.7" y="177.8" radius="4.5085" width="0.2032" layer="16"/>
+<circle x="12.7" y="355.6" radius="4.5085" width="0.2032" layer="16"/>
+<circle x="419.1" y="355.6" radius="4.5085" width="0.2032" layer="16"/>
+<circle x="419.1" y="177.8" radius="4.5085" width="0.2032" layer="16"/>
+<circle x="419.1" y="0" radius="4.5085" width="0.2032" layer="16"/>
+<wire x1="30.48" y1="-3.81" x2="30.48" y2="358.14" width="0.2032" layer="21"/>
+<wire x1="30.48" y1="358.14" x2="45.72" y2="358.14" width="0.2032" layer="21" curve="-159.222284"/>
+<wire x1="45.72" y1="358.14" x2="45.72" y2="-3.81" width="0.2032" layer="21"/>
+<wire x1="45.72" y1="-3.81" x2="30.48" y2="-3.81" width="0.2032" layer="21" curve="-159.222284"/>
+<wire x1="411.48" y1="-3.81" x2="426.72" y2="-3.81" width="0.2032" layer="21" curve="159.222284"/>
+<wire x1="426.72" y1="-3.81" x2="426.72" y2="358.14" width="0.2032" layer="21"/>
+<wire x1="426.72" y1="358.14" x2="411.48" y2="358.14" width="0.2032" layer="21" curve="159.222284"/>
+<wire x1="411.48" y1="358.14" x2="411.48" y2="-3.81" width="0.2032" layer="21"/>
+<circle x="127" y="177.8" radius="4.5085" width="0.2032" layer="21"/>
+<circle x="127" y="355.6" radius="4.5085" width="0.2032" layer="21"/>
+<circle x="304.8" y="355.6" radius="4.5085" width="0.2032" layer="21"/>
+<circle x="304.8" y="177.8" radius="4.5085" width="0.2032" layer="21"/>
+<circle x="304.8" y="0" radius="4.5085" width="0.2032" layer="21"/>
+<circle x="127" y="0" radius="4.5085" width="0.2032" layer="21"/>
 </plain>
 <attributes>
@@
 <signals>
 <signal name="S$1">
-<wire x1="20.32" y1="-3.81" x2="20.32" y2="358.14" width="0.2032" layer="16"/>
-<wire x1="20.32" y1="358.14" x2="5.08" y2="358.14" width="0.2032" layer="16" curve="159.222284"/>
-<wire x1="5.08" y1="358.14" x2="5.08" y2="-3.81" width="0.2032" layer="16"/>
-<wire x1="5.08" y1="-3.81" x2="20.32" y2="-3.81" width="0.2032" layer="16" curve="159.222284"/>
-</signal>
-<signal name="S$2">
-<wire x1="45.72" y1="-3.81" x2="45.72" y2="358.14" width="0.2032" layer="16"/>
-<wire x1="45.72" y1="358.14" x2="30.48" y2="358.14" width="0.2032" layer="16" curve="159.222284"/>
-<wire x1="30.48" y1="358.14" x2="30.48" y2="-3.81" width="0.2032" layer="16"/>
-<wire x1="30.48" y1="-3.81" x2="45.72" y2="-3.81" width="0.2032" layer="16" curve="159.222284"/>
+<wire x1="20.32" y1="-3.81" x2="20.32" y2="358.14" width="0.2032" layer="1"/>
+<wire x1="20.32" y1="358.14" x2="5.08" y2="358.14" width="0.2032" layer="1" curve="159.222284"/>
+<wire x1="5.08" y1="358.14" x2="5.08" y2="-3.81" width="0.2032" layer="1"/>
+<wire x1="5.08" y1="-3.81" x2="20.32" y2="-3.81" width="0.2032" layer="1" curve="159.222284"/>
 </signal>
 <signal name="S$3">
-<wire x1="401.32" y1="-3.81" x2="401.32" y2="358.14" width="0.2032" layer="16"/>
-<wire x1="401.32" y1="358.14" x2="386.08" y2="358.14" width="0.2032" layer="16" curve="159.222284"/>
-<wire x1="386.08" y1="358.14" x2="386.08" y2="-3.81" width="0.2032" layer="16"/>
-<wire x1="386.08" y1="-3.81" x2="401.32" y2="-3.81" width="0.2032" layer="16" curve="159.222284"/>
-</signal>
-<signal name="S$4">
-<wire x1="426.72" y1="-3.81" x2="426.72" y2="358.14" width="0.2032" layer="16"/>
-<wire x1="426.72" y1="358.14" x2="411.48" y2="358.14" width="0.2032" layer="16" curve="159.222284"/>
-<wire x1="411.48" y1="358.14" x2="411.48" y2="-3.81" width="0.2032" layer="16"/>
-<wire x1="411.48" y1="-3.81" x2="426.72" y2="-3.81" width="0.2032" layer="16" curve="159.222284"/>
+<wire x1="401.32" y1="-3.81" x2="401.32" y2="358.14" width="0.2032" layer="1"/>
+<wire x1="401.32" y1="358.14" x2="386.08" y2="358.14" width="0.2032" layer="1" curve="159.222284"/>
+<wire x1="386.08" y1="358.14" x2="386.08" y2="-3.81" width="0.2032" layer="1"/>
+<wire x1="386.08" y1="-3.81" x2="401.32" y2="-3.81" width="0.2032" layer="1" curve="159.222284"/>
 </signal>
 <signal name="S$5">
