File: cap.brd (EAGLE design)
At the start: 25.4 x 30.5 mm, 5 parts

Commit message: confirm footprints and finalize for maker faire
Parts:
- removed E$6: (no value), tekdemo:PANASONIC_C
- moved E$5 3.81 mm to (12.7, 16.3)
- moved E$1 2.03 mm to (12.7, 20.8)
- moved E$2 2.03 mm to (12.7, 23.4)
Routing:
- net S$3: track 28.6 -> 26.9 mm, vias 1 -> 2
- net S$6: track 25.8 -> 24.5 mm, vias 0 -> 1
- added copper zone on layer 16, net S$5
- added copper zone on layer 1, net S$7
Other:
- board text removed: "d"
- board text removed: "g"
- board text removed: "s"
